File: Transmitter/Transmitter loadsharing/Transmitter loadsharing.kicad_sch (KiCad schematic)
At the start: 115 parts, among them J1 Conn_Coaxial, J10 Conn_01x01, J11 Conn_01x01, J12 Conn_01x01, J13 Conn_01x01, J14 Conn_01x01, J15 Conn_01x01, J16 Conn_01x01, J17 Conn_Coaxial, J18 Conn_Coaxial, J19 Conn_Coaxial, J2 Conn_01x03, J20 Conn_01x01, J21 Conn_01x01, J22 Conn_01x01, J23 Conn_01x01, J24 Conn_01x01, J25 Conn_01x01, J3 Conn_01x03, J4 Conn_01x02_Socket, J5 Conn_01x02, J6 Conn_01x01, J7 Conn_01x02, J8 Conn_01x02_Socket Horizontal, J9 Conn_01x01, U1 OPA3692IDBQR, U10 LT3094EMSE-PBF, U11 LT3094EMSE-PBF, U2 THS3091D, U3 THS3091D, U4 THS3091D, U5 THS3091D, U6 THS3091D, U7 THS3091D, U8 LT3045EMSE-PBF, U9 LT3045EMSE-PBF

Commit message: added LTM8049 symbol/footprint
Parts:
- J17, J18: footprint Connector_Coaxial:BNC_Amphenol_B6252HB-NPP3G-50_Horizontal -> BNc_Amphenol_112640:BNC_Amphenol_112640_Edge_mount
Changed lines of the file:
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@@
 			)
 		)
-		(property "Footprint" "Connector_Coaxial:BNC_Amphenol_B6252HB-NPP3G-50_Horizontal"
+		(property "Footprint" "BNc_Amphenol_112640:BNC_Amphenol_112640_Edge_mount"
 			(at 320.04 21.59 0)
 			(effects
@@
 			)
 		)
-		(property "Footprint" "Connector_Coaxial:BNC_Amphenol_B6252HB-NPP3G-50_Horizontal"
+		(property "Footprint" "BNc_Amphenol_112640:BNC_Amphenol_112640_Edge_mount"
 			(at 233.68 20.32 0)
 			(effects

Commit message: not enough room?
Parts:
- added C38, C43: 4.7u, Capacitor_SMD:C_0603_1608Metric_Pad1.08x0.95mm_HandSolder, symbol Device:C
- added C39: 0.47u, Capacitor_SMD:C_0603_1608Metric_Pad1.08x0.95mm_HandSolder, symbol Device:C
- added C40, C41, C42: 10u, Capacitor_SMD:C_0603_1608Metric_Pad1.08x0.95mm_HandSolder, symbol Device:C
- added J26: Conn_Coaxial, BNc_Amphenol_112640:BNC_Amphenol_112640_Edge_mount, symbol Connector:Conn_Coaxial
- added J27, J28: Conn_01x01, Connector_PinHeader_2.54mm:PinHeader_1x01_P2.54mm_Vertical, symbol Connector_Generic:Conn_01x01
- added R43, R46: 49.9k, Resistor_SMD:R_0603_1608Metric_Pad0.98x0.95mm_HandSolder, symbol Device:R
- added U13: LT3045EMSE-PBF, LT3045:MSOP12_MSE_ADI, symbol LT3045 MSOP:LT3045EMSE-PBF
- added U14: LT3094EMSE-PBF, LT3094:05-08-1666_ADI, symbol LT3094 MSOP:LT3094EMSE-PBF
- R40, R41: value 24.9k -> 150k
Connections:
- net +5V: now also C40.1, U13.10 (OUTS), U13.11 (OUT), U13.12 (OUT); no longer C13.2, C15.2, C17.2, C23.2, C24.2, C25.2, C27.1, C28.1, U2.7 (VS+), U3.7 (VS+), U4.7 (VS+), U5.7 (VS+), U6.7 (VS+), U7.7 (VS+), U8.10 (OUTS), U8.11 (OUT), U8.12 (OUT), U9.10 (OUTS), U9.11 (OUT), U9.12 (OUT)
- net -5V: now also C42.1, U14.10 (OUTS), U14.11 (OUT), U14.12 (OUT); no longer C11.1, C12.1, C16.1, C19.1, C20.1, C21.1, C31.1, C32.1, U10.10 (OUTS), U10.11 (OUT), U10.12 (OUT), U11.10 (OUTS), U11.11 (OUT), U11.12 (OUT), U2.4 (VS-), U3.4 (VS-), U4.4 (VS-), U5.4 (VS-), U6.4 (VS-), U7.4 (VS-)
- net GND: now also C38.2, C39.2, C40.2, C41.2, C42.2, C43.2, J26.2 (Ext), J28.1 (Pin_1), R43.2, R46.2, U13.6 (ILIM), U13.9 (GND), U13.EPAD (GND), U14.6 (ILIM), U14.9 (GND)
- net PWR+: now also C38.1, U13.1 (IN), U13.2 (IN), U13.3 (IN), U13.4 (EN/UV), U13.7 (PGFB); no longer C9.1, U8.1 (IN), U8.2 (IN), U8.3 (IN), U8.4 (EN/UV), U8.7 (PGFB), U9.1 (IN), U9.2 (IN), U9.3 (IN), U9.4 (EN/UV), U9.7 (PGFB)
- net PWR-: now also C41.1, U14.1 (IN), U14.13 (IN), U14.2 (IN), U14.3 (EN/UV), U14.5 (PGFB); no longer C29.1, U10.1 (IN), U10.13 (IN), U10.2 (IN), U10.3 (EN/UV), U10.5 (PGFB), U11.1 (IN), U11.13 (IN), U11.2 (IN), U11.3 (EN/UV), U11.5 (PGFB)
- new net: C43.1, R46.1, U14.8 (SET)
- new net: C39.1, R43.1, U13.8 (SET)
- new net +15V: C13.2, C15.2, C17.2, C23.2, C24.2, C25.2, U2.7 (VS+), U3.7 (VS+), U4.7 (VS+), U5.7 (VS+), U6.7 (VS+), U7.7 (VS+)
- new net +15V_In: C27.1, C28.1, U8.10 (OUTS), U8.11 (OUT), U8.12 (OUT), U9.10 (OUTS), U9.11 (OUT), U9.12 (OUT)
- new net -15V: C11.1, C12.1, C16.1, C19.1, C20.1, C21.1, U2.4 (VS-), U3.4 (VS-), U4.4 (VS-), U5.4 (VS-), U6.4 (VS-), U7.4 (VS-)
- new net -15V_In: C31.1, C32.1, U10.10 (OUTS), U10.11 (OUT), U10.12 (OUT), U11.10 (OUTS), U11.11 (OUT), U11.12 (OUT)
- new net LTM8049 Sheet/+15V: C9.1, U8.1 (IN), U8.2 (IN), U8.3 (IN), U8.4 (EN/UV), U8.7 (PGFB), U9.1 (IN), U9.2 (IN), U9.3 (IN), U9.4 (EN/UV), U9.7 (PGFB)
- new net LTM8049 Sheet/-15V: C29.1, U10.1 (IN), U10.13 (IN), U10.2 (IN), U10.3 (EN/UV), U10.5 (PGFB), U11.1 (IN), U11.13 (IN), U11.2 (IN), U11.3 (EN/UV), U11.5 (PGFB)
- new net LTM8049 Sheet/Vin: J26.1 (In), J27.1 (Pin_1)
- no-connect marks 29 -> 32
Other:
- added sheet LTM8049 Sheet (LTM8049.kicad_sch)
- note added: "+15V regulator circut"
- title: (none) -> Transmitter
- moved on the sheet: C10, C11, C12, C13, C14, C15, C16, C17, C18, C19, C20, C21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
