File: Transmitter/Transmitter loadsharing/Transmitter loadsharing.kicad_pcb (KiCad board)
At the start: 4 copper layers, 145 x 50.8 mm, 115 parts, among them J1 Conn_Coaxial, J10 Conn_01x01, J11 Conn_01x01, J12 Conn_01x01, J13 Conn_01x01, J14 Conn_01x01, J15 Conn_01x01, J16 Conn_01x01, J17 Conn_Coaxial, J18 Conn_Coaxial, J19 Conn_Coaxial, J2 Conn_01x03, J20 Conn_01x01, J21 Conn_01x01, J22 Conn_01x01, J23 Conn_01x01, J24 Conn_01x01, J25 Conn_01x01, J3 Conn_01x03, J4 Conn_01x02_Socket, J5 Conn_01x02, J6 Conn_01x01, J7 Conn_01x02, J8 Conn_01x02_Socket Horizontal, J9 Conn_01x01, U1 OPA3692IDBQR, U10 LT3094EMSE-PBF, U11 LT3094EMSE-PBF, U2 THS3091D, U3 THS3091D, U4 THS3091D, U5 THS3091D, U6 THS3091D, U7 THS3091D, U8 LT3045EMSE-PBF, U9 LT3045EMSE-PBF

Commit message: Final version before review 3
Parts:
- U1: footprint Opa3692 SOIC:DBQ16 -> Opa3692 SSOP:DBQ16
- moved H1 0.63 mm to (91.0, 54.2)
- moved H2 0.63 mm to (91.0, 96.5)
- moved H3 0.42 mm to (227.6, 96.5)
- moved H4 0.42 mm to (227.6, 54.2)
Other:
- outline, holes or cut-outs redrawn
- board text added: "Transmitter 1.1 2024-05-2"
- board text removed: "Transmitter 1.1 2024-04-19"
Changed lines of the file:
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@@
 			)
 		)
+		(property ki_fp_filters "*BNC* *SMA* *SMB* *SMC* *Cinch* *LEMO* *UMRF* *MCX* *U.FL*")
+		(sheetname "Root")
+		(sheetfile "Transmitter loadsharing.kicad_sch")
 		(fp_line
 			(start -1.24 0.27)
@@
 		)
 		(group ""
-			(members "0d9544db-5788-496f-a1b6-a4c34ec4e949" "737e8321-c275-4ee5-bd18-455d36bb17f3"
-				"d12421bc-9db6-49de-8399-16b6aafa9bce"
+			(members "19f5e964-bab6-4cd2-b0ef-c114dd5d8577" "54c97a73-ad56-4140-a55a-7d7a97c31070"
+				"7b8cf88b-1e53-4819-975f-0048b4d83672"
 			)
 		)
 		(group ""
-			(members "251dce33-2187-452d-a227-155de697e610" "add2e8ac-c621-4877-9947-3e0b8e4962b9")
-		)
-		(model "C:/Projects/KiCad/Spiral/Kicad Degree project GIT/Degree-Project-KiCad/BNc_Amphenol_112640.pretty/112640.stp"
-			(offset
-				(xyz 0 0 0.3)
-			)
-			(scale
-				(xyz 1 1 1)
-			)
-			(rotate
-				(xyz 0 -90 90)
-			)
+			(members "bfe1ad41-815c-4f59-91e9-7a53ea157324" "fe37fb25-6936-4d12-9a4e-3b1022e88fad")
 		)
 	)
-	(footprint "Opa3692 SOIC:DBQ16"
+	(footprint "Opa3692 SSOP:DBQ16"
 		(layer "F.Cu")
 		(at 128.3125 92.233348 90)
@@
 			)
 		)
-		(property "Footprint" "Opa3692 SOIC:DBQ16"
+		(property "Footprint" "Opa3692 SSOP:DBQ16"
 			(at 0 0 90)
 			(unlocked yes)
@@
 			(layer "F.Fab")
 		)
+		(fp_text user "*"
+			(at -2.8067 -3.7211 90)
+			(layer "F.SilkS")
+			(effects
+				(font
+					(size 1 1)
+					(thickness 0.15)
+				)
+			)
+		)
 		(fp_text user "${REFERENCE}"
 			(at 0 0 90)
@@
 			)
 		)
+		(fp_text user "*"
+			(at -2.8067 -3.7211 90)
+			(layer "F.Fab")
+			(effects
+				(font
+					(size 1 1)
+					(thickness 0.15)
+				)
+			)
+		)
+		(fp_text user "*"
+			(at -2.8067 -3.7211 90)
+			(unlocked yes)
+			(layer "F.Fab")
+			(effects
+				(font
+					(size 1 1)
+					(thickness 0.15)
+				)
+			)
+		)
 		(pad "1" smd rect
 			(at -2.5527 -2.2225 90)
@@
 			(pintype "unspecified+no_connect")
 		)
-		(model "C:/Projects/KiCad/Spiral/Kicad Degree project GIT/Degree-Project-KiCad/OPA3692/R/DBQ0016A.stp"
-			(offset
-				(xyz 0 0 1)
-			)
-			(scale
-				(xyz 1 1 1)
-			)
-			(rotate
-				(xyz -90 0 90)
-			)
-		)
 	)
 	(footprint "Resistor_SMD:R_0603_1608Metric_Pad0.98x0.95mm_HandSolder"
@@
 			)
 		)
+		(property ki_fp_filters "*BNC* *SMA* *SMB* *SMC* *Cinch* *LEMO* *UMRF* *MCX* *U.FL*")
+		(sheetname "Root")
+		(sheetfile "Transmitter loadsharing.kicad_sch")
 		(fp_line
 			(start -1.24 0.27)
@@
 		)
 		(group ""
-			(members "24d62238-16e9-4b54-b5f4-5e42fc941801" "3221d079-a4d5-4f61-9ce2-6772b3de6d95"
-				"cacbf135-269c-4325-8ebc-44a5d89c0001"
+			(members "00efdfaf-0666-4cf2-ad88-e8e6e47144c9" "2edb6283-76c1-4103-8dbd-15ef8bef704b"
+				"435e3baa-30e3-4501-a730-e154bf7e512c"
 			)
 		)
 		(group ""
-			(members "76805bd4-a0b3-43e5-a265-6cf97f1df7a1" "b5b07520-167d-4d53-936a-f3b17ab15a43")
-		)
-		(model "C:/Projects/KiCad/Spiral/Kicad Degree project GIT/Degree-Project-KiCad/BNc_Amphenol_112640.pretty/112640.stp"
-			(offset
-				(xyz 0 0 0.3)
-			)
-			(scale
-				(xyz 1 1 1)
-			)
-			(rotate
-				(xyz 0 -90 90)
-			)
+			(members "8d29b2e1-234f-4fa8-a14b-239c7b0fb0de" "913cab1d-2a60-4061-a49d-f74d3c4b7023")
 		)
 	)
@@
 	(footprint "MountingHole:MountingHole_3.2mm_M3_Pad"
 		(layer "F.Cu")
-		(at 91.5 54.5)
+		(at 90.95 54.2)
 		(descr "Mounting Hole 3.2mm, M3")
 		(tags "mounting hole 3.2mm m3")
@@
 	(footprint "MountingHole:MountingHole_3.2mm_M3_Pad"
 		(layer "F.Cu")
-		(at 227.25 54.5)
+		(at 227.55 54.2)
 		(descr "Mounting Hole 3.2mm, M3")
 		(tags "mounting hole 3.2mm m3")
@@
 	(footprint "MountingHole:MountingHole_3.2mm_M3_Pad"
 		(layer "F.Cu")
-		(at 91.5 96.25)
+		(at 90.95 96.55)
 		(descr "Mounting Hole 3.2mm, M3")
 		(tags "mounting hole 3.2mm m3")
@@
 	(footprint "MountingHole:MountingHole_3.2mm_M3_Pad"
 		(layer "F.Cu")
-		(at 227.25 96.25)
+		(at 227.55 96.55)
 		(descr "Mounting Hole 3.2mm, M3")
 		(tags "mounting hole 3.2mm m3")
@@
 		)
 	)
-	(gr_rect
-		(start 86.75 50)
-		(end 231.75 100.75)
+	(gr_line
+		(start 86.75 96.55)
+		(end 86.75 54.2)
+		(stroke
+			(width 0.05)
+			(type default)
+		)
+		(layer "Edge.Cuts")
+	)
+	(gr_line
+		(start 227.55 100.75)
+		(end 90.95 100.75)
+		(stroke
+			(width 0.05)
+			(type default)
+		)
+		(layer "Edge.Cuts")
+	)
+	(gr_arc
+		(start 231.750011 96.55)
+		(mid 230.519856 99.519856)
+		(end 227.55 100.750011)
+		(stroke
+			(width 0.05)
+			(type default)
+		)
+		(layer "Edge.Cuts")
+	)
+	(gr_arc
+		(start 86.749703 54.2)
+		(mid 87.979942 51.229942)
+		(end 90.95 49.999703)
+		(stroke
+			(width 0.05)
+			(type default)
+		)
+		(layer "Edge.Cuts")
+	)
+	(gr_line
+		(start 231.75 96.55)
+		(end 231.75 54.2)
+		(stroke
+			(width 0.05)
+			(type default)
+		)
+		(layer "Edge.Cuts")
+	)
+	(gr_arc
+		(start 90.95 100.750297)
+		(mid 87.979942 99.520058)
+		(end 86.749703 96.55)
+		(stroke
+			(width 0.05)
+			(type default)
+		)
+		(layer "Edge.Cuts")
+	)
+	(gr_line
+		(start 227.55 50)
+		(end 90.95 50)
+		(stroke
+			(width 0.05)
+			(type default)
+		)
+		(layer "Edge.Cuts")
+	)
+	(gr_arc
+		(start 227.55 49.999953)
+		(mid 230.519882 51.230118)
+		(end 231.750047 54.2)
 		(stroke
 			(width 0.05)
 			(type default)
 		)
-		(fill none)
 		(layer "Edge.Cuts")
 	)
-	(gr_text "Transmitter 1.1 2024-04-19"
+	(gr_text "Transmitter 1.1 2024-05-2\n"
 		(at 229.4888 63.8726 90)
 		(layer "B.SilkS")
@@
 		(layer "User.1")
 		(pts
-			(xy 231.75 100.75) (xy 86.75 100.75)
+			(xy 86.75 96.55) (xy 231.750011 96.55)
 		)
-		(height -21.35)
+		(height 37.81)
 		(gr_text "145.0000 mm"
-			(at 159.25 126.2226 0)
+			(at 159.250006 133.21 0)
 			(layer "User.1")
 			(effects
@@
 			(thickness 0.1)
 			(arrow_length 1.27)
-			(text_position_mode 2)
+			(text_position_mode 0)
 			(extension_height 0.58642)
 			(extension_offset 0.5) keep_text_aligned)
@@
 		(layer "User.1")
 		(pts
-			(xy 86.75 50) (xy 86.75 100.75)
+			(xy 90.95 50) (xy 90.95 100.75)
 		)
-		(height 24.575)
+		(height 27.01)
 		(gr_text "50.7500 mm"
-			(at 61.025 75.375 90)
+			(at 62.79 75.375 90)
 			(layer "User.1")
 			(effects

Commit message: blurp
Parts:
- C30: value 0.47uF -> 4.7uF
Changed lines of the file:
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@@
 			)
 		)
-		(property "Value" "0.47uF"
+		(property "Value" "4.7uF"
 			(at 3.8375 0.1 90)
 			(layer "F.Fab")
